File: DacAmp/usb.kicad_sch (KiCad schematic)
At the start: 0 parts

Commit message: add usb + codec
Parts:
- added C2: 2n2, Capacitor_SMD:C_0805_2012Metric_Pad1.18x1.45mm_HandSolder, symbol Device:C_Small
- added D1, D2: ESD321, ESD321DYAR:SOT5x3_DYA_TEX-M, symbol ESD321DYAR:ESD321DYAR
- added J2: USB_B, Connector_USB:USB_B_OST_USB-B1HSxx_Horizontal, symbol Connector:USB_B
- added R2: DNP, Resistor_SMD:R_0402_1005Metric_Pad0.72x0.64mm_HandSolder, symbol Device:R_Small_US
Connections:
- new net CGND: C2.1, J2.5 (Shield), R2.1
- new net CONN_D+: D2.2, J2.3 (D+)
- new net CONN_D-: D1.2, J2.2 (D-)
- new net GND: C2.2, D1.1, D2.1, J2.4 (GND), R2.2
- new net VUSB_CONN: J2.1 (VBUS)
Other:
- note added: "1kV"
- note added: "choose HV rating cap:"
