File: DacAmp/usb.kicad_sch (KiCad schematic)
At the start: 5 parts, among them J2 USB_B

Commit message: add components and footprints
Parts:
- removed D1, D2: ESD321, ESD321DYAR:SOT5x3_DYA_TEX-M, symbol ESD321DYAR:ESD321DYAR
- added D1, D2: ESD321, ul_ESD321DYAR:SOT5x3_DYA_TEX-M, symbol 2024-10-02_15-56-16:ESD321DYAR
Connections:
- net CONN_D+: now also D2.2
- net CONN_D-: now also D1.2
- net GND: now also D1.1, D2.1
Changed lines of the file:
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@@
+	)
+	(symbol
+		(lib_id "2024-10-02_15-56-16:ESD321DYAR")
+		(at 77.47 80.01 90)
+		(unit 1)
+		(exclude_from_sim no)
+		(in_bom yes)
+		(on_board yes)
+		(dnp no)
+		(fields_autoplaced yes)
+		(property "Reference" "D2"
+			(at 81.28 73.6599 90)
+			(effects
+				(font
+					(size 1.524 1.524)
+				)
+				(justify right)
+			)
+		)
+		(property "Value" "ESD321"
+			(at 81.28 76.1999 90)
+			(effects
+				(font
+					(size 1.524 1.524)
+				)
+				(justify right)
+			)
+		)
+		(property "Footprint" "ul_ESD321DYAR:SOT5x3_DYA_TEX-M"
+			(at 77.47 80.01 0)
+			(effects
+				(font
+					(size 1.27 1.27)
+					(italic yes)
+				)
+				(hide yes)
+			)
+		)
+		(property "Datasheet" "ESD321DYAR"
+			(at 77.47 80.01 0)
+			(effects
+				(font
+					(size 1.27 1.27)
+					(italic yes)
+				)
+				(hide yes)
+			)
+		)
+		(property "Description" ""
+			(at 77.47 80.01 0)
+			(effects
+				(font
+					(size 1.27 1.27)
+				)
+				(hide yes)
+			)
+		)
+		(pin "2"
+		)
+		(pin "1"
+		)
+		(instances
+			(project "DacAmp"
+				(path "/d6da33f4-6bef-4098-a08b-0ea38da216b8/444411ed-867e-42ae-9836-72e43d6ad6a6"
+					(reference "D2")
+					(unit 1)
+				)
+			)
+		)
 	)
 	(symbol
@@
 				(path "/d6da33f4-6bef-4098-a08b-0ea38da216b8/444411ed-867e-42ae-9836-72e43d6ad6a6"
 					(reference "J2")
-					(unit 1)
-				)
-			)
-		)
-	)
-	(symbol
-		(lib_id "ESD321DYAR:ESD321DYAR")
-		(at 59.69 80.01 90)
-		(unit 1)
-		(exclude_from_sim no)
-		(in_bom yes)
-		(on_board yes)
-		(dnp no)
-		(fields_autoplaced yes)
-		(property "Reference" "D1"
-			(at 63.5 73.6599 90)
-			(effects
-				(font
-					(size 1.524 1.524)
-				)
-				(justify right)
-			)
-		)
-		(property "Value" "ESD321"
-			(at 63.5 76.1999 90)
-			(effects
-				(font
-					(size 1.524 1.524)
-				)
-				(justify right)
-			)
-		)
-		(property "Footprint" "ESD321DYAR:SOT5x3_DYA_TEX-M"
-			(at 59.69 80.01 0)
-			(effects
-				(font
-					(size 1.27 1.27)
-					(italic yes)
-				)
-				(hide yes)
-			)
-		)
-		(property "Datasheet" "ESD321DYAR"
-			(at 59.69 80.01 0)
-			(effects
-				(font
-					(size 1.27 1.27)
-					(italic yes)
-				)
-				(hide yes)
-			)
-		)
-		(property "Description" ""
-			(at 59.69 80.01 0)
-			(effects
-				(font
-					(size 1.27 1.27)
-				)
-				(hide yes)
-			)
-		)
-		(property "Field5" ""
-			(at 59.69 80.01 0)
-			(effects
-				(font
-					(size 1.27 1.27)
-				)
-				(hide yes)
-			)
-		)
-		(pin "2"
-		)
-		(pin "1"
-		)
-		(instances
-			(project "DacAmp"
-				(path "/d6da33f4-6bef-4098-a08b-0ea38da216b8/444411ed-867e-42ae-9836-72e43d6ad6a6"
-					(reference "D1")
 					(unit 1)
 				)
@@
 	)
 	(symbol
-		(lib_id "ESD321DYAR:ESD321DYAR")
-		(at 77.47 80.01 90)
-		(unit 1)
-		(exclude_from_sim no)
-		(in_bom yes)
-		(on_board yes)
-		(dnp no)
-		(fields_autoplaced yes)
-		(property "Reference" "D2"
-			(at 81.28 73.6599 90)
+		(lib_id "2024-10-02_15-56-16:ESD321DYAR")
+		(at 59.69 80.01 90)
+		(unit 1)
+		(exclude_from_sim no)
+		(in_bom yes)
+		(on_board yes)
+		(dnp no)
+		(fields_autoplaced yes)
+		(property "Reference" "D1"
+			(at 63.5 73.6599 90)
 			(effects
 				(font
@@
 		)
 		(property "Value" "ESD321"
-			(at 81.28 76.1999 90)
+			(at 63.5 76.1999 90)
 			(effects
 				(font
@@
 			)
 		)
-		(property "Footprint" "ESD321DYAR:SOT5x3_DYA_TEX-M"
-			(at 77.47 80.01 0)
+		(property "Footprint" "ul_ESD321DYAR:SOT5x3_DYA_TEX-M"
+			(at 59.69 80.01 0)
 			(effects
 				(font
@@
 		)
 		(property "Datasheet" "ESD321DYAR"
-			(at 77.47 80.01 0)
+			(at 59.69 80.01 0)
 			(effects
 				(font
@@
 		)
 		(property "Description" ""
-			(at 77.47 80.01 0)
-			(effects
-				(font
-					(size 1.27 1.27)
-				)
-				(hide yes)
-			)
-		)
-		(property "Field5" ""
-			(at 77.47 80.01 0)
+			(at 59.69 80.01 0)
 			(effects
 				(font
@@
 		)
 		(instances
-			(project "DacAmp"
-				(path "/d6da33f4-6bef-4098-a08b-0ea38da216b8/444411ed-867e-42ae-9836-72e43d6ad6a6"
-					(reference "D2")
-					(unit 1)
-				)
+			(project ""
+				(path "/d6da33f4-6bef-4098-a08b-0ea38da216b8/444411ed-867e-42ae-9836-72e43d6ad6a6"
+					(reference "D1")
+					(unit 1)
+				)

Commit message: component placement for op amps
Parts:
- added C39: 100n, Capacitor_SMD:C_0402_1005Metric_Pad0.74x0.62mm_HandSolder, symbol Device:C
- added C40: 10n, Capacitor_SMD:C_0402_1005Metric_Pad0.74x0.62mm_HandSolder, symbol Device:C
- added FB1: BLM18PG221SN1D, Inductor_SMD:L_0603_1608Metric_Pad1.05x0.95mm_HandSolder, symbol Device:FerriteBead
- added TP5, TP6: TestPoint, TestPoint:TestPoint_Pad_D1.5mm, symbol Connector:TestPoint
Connections:
- net GND: now also C39.2, C40.2
- net VUSB_CONN: now also C40.1, FB1.1, TP6.1
- new net VBUS: C39.1, FB1.2, TP5.1
