File: DacAmp/DacAmp.kicad_sch (KiCad schematic)
At the start: 0 parts

Commit message: finish rough floor plan
Parts:
- added H1, H2, H3, H4: MountingHole_Pad, MountingHole:MountingHole_2.7mm_M2.5_ISO7380_Pad, symbol Mechanical:MountingHole_Pad
Connections:
- new net GND: H1.1, H2.1, H3.1, H4.1
