File: DacAmp/power.kicad_sch (KiCad schematic)
At the start: 0 parts

Commit message: complete overall schematic, TODO: find values and add net labels
Parts:
- added C21, C22, C24: 1u, Capacitor_SMD:C_0402_1005Metric_Pad0.74x0.62mm_HandSolder, symbol Device:C_Small
- added C26: 10u, Capacitor_SMD:C_0805_2012Metric_Pad1.18x1.45mm_HandSolder, symbol Device:C
- added C27: 100u, symbol Device:C_Polarized_US
- added C28: 100n, symbol Device:C
- added L1: L, symbol Device:L
- added R27, R29, R30, R31: R_US, symbol Device:R_US
- added R32, R33: 1R, symbol Device:R_US
- added TP1, TP2, TP3: TestPoint, symbol Connector:TestPoint
- added U10: TLV70237_SOT23-5, Package_TO_SOT_SMD:SOT-23-5, symbol Regulator_Linear:TLV70237_SOT23-5
- added U11: TLV61046ADB, Package_TO_SOT_SMD:SOT-23-6, symbol Regulator_Switching:TLV61046ADB
- added U12: NE5532, Package_SO:SOIC-8_3.9x4.9mm_P1.27mm, symbol Amplifier_Operational:NE5532
Connections:
- new net: C27.1, R30.2, R31.1, U12.3 (+), U12.5 (+)
- new net: R32.1, U12.1, U12.2 (-)
- new net: R27.2, R29.1, U11.3 (FB)
- new net: L1.2, U11.1 (SW)
- new net: R33.1, U12.6 (-), U12.7
- new net 15V: C26.1, C28.1, R27.1, R30.1, TP2.1, U11.5 (VOUT), U12.8 (V+)
- new net 3V7: C22.1, TP1.1, U10.5 (OUT)
- new net 7V5: R32.2, R33.2, TP3.1
- new net GND: C21.2, C22.2, C24.2, C26.2, C27.2, C28.2, R29.2, R31.2, U10.2 (GND), U11.2 (GND), U12.4 (V-)
- new net VBUS: C21.1, C24.1, L1.1, U10.1 (IN), U10.3 (EN), U11.4 (EN), U11.6 (VI)
Other:
- note added: "15V @ 100mA Boost Converter"
- note added: "3V7 @ 300 mA LDO"
- note added: "Half-rail bias generator"
- note added: "derate"

Commit message: add 15v LDO
Parts:
- removed C21: 1u, Capacitor_SMD:C_0402_1005Metric_Pad0.74x0.62mm_HandSolder, symbol Device:C_Small
- added C21: 100n, Capacitor_SMD:C_0402_1005Metric_Pad0.74x0.62mm_HandSolder, symbol Device:C
- added C37: 22u, symbol Device:C_Polarized_US
- added C38: 1u, Capacitor_SMD:C_0805_2012Metric_Pad1.18x1.45mm_HandSolder, symbol Device:C
- added R34: 10k7, symbol Device:R_US
- added R35: 1k, symbol Device:R_US
- added TP4: TestPoint, symbol Connector:TestPoint
- added U13: LM2941LD_NOPB, LM2941:DFN400X400X80-9N, symbol LM2941:LM2941LD_NOPB
- C22: value 1u -> 4u7
- C26: footprint Capacitor_SMD:C_0805_2012Metric_Pad1.18x1.45mm_HandSolder -> Capacitor_SMD:C_1210_3225Metric_Pad1.33x2.70mm_HandSolder
- C28: footprint (none) -> Capacitor_SMD:C_0805_2012Metric_Pad1.18x1.45mm_HandSolder
Connections:
- net 15V: now also C37.1, R34.1, TP4.1, U13.5 (OUT); no longer C26.1, R27.1, TP2.1, U11.5 (VOUT)
- net GND: now also C21.2, C37.2, C38.2, R35.2, U13.2 (GND), U13.7 (GND), U13.9 (GND)
- net VBUS: now also C21.1
- new net 17V: C26.1, C38.1, R27.1, TP2.1, U11.5 (VOUT), U13.1 (EN), U13.3 (IN)
- new net ADJ: R34.2, R35.1, U13.8 (ADJ)
Other:
- note added: "Boost Converter (17V @ 100mA)"
- note added: "LDO (15V @ 1A)"
- note added: "LDO (3V7 @ 300 mA)"
- note added: "VOUT = 1.275 × ((R1 + R2) / R1) = 14.9175V"
- note removed: "15V @ 100mA Boost Converter"
- note removed: "3V7 @ 300 mA LDO"
- note removed: "derate"
- moved on the sheet: C27, C28, R30, R31, R32, R33, TP3, U12A, U12B, U12C

Commit message: add inductor value 10uH
Parts:
- L1: value L -> 10u
Other:
- note added: "prob just put a 10u here or something."
Changed lines of the file:
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@@
+		)
+	)
+	(text "prob just put a 10u here or something."
+		(exclude_from_sim no)
+		(at 76.454 62.23 0)
+		(effects
+			(font
+				(size 1.27 1.27)
+			)
 		)
 	)
@@
 			)
 		)
-		(property "Value" "L"
+		(property "Value" "10u"
 			(at 127 27.94 90)
 			(effects

Commit message: add footprints to almost everything
Parts:
- C27: footprint (none) -> Capacitor_THT:CP_Radial_D8.0mm_P3.50mm
- L1: value 10u -> 10uH
- R30, R31: value R_US -> 20k; footprint (none) -> Resistor_SMD:R_0402_1005Metric_Pad0.72x0.64mm_HandSolder
- R32, R33: footprint (none) -> Resistor_SMD:R_0603_1608Metric_Pad0.98x0.95mm_HandSolder
- TP1, TP2, TP3, TP4: footprint (none) -> TestPoint:TestPoint_Pad_D1.5mm
Connections:
- net 15V: now also R30.2; no longer R30.1
- net GND: now also R31.1; no longer R31.2
- net at C27.1, U12.3 (+), U12.5 (+): now also R30.1, R31.2; no longer R30.2, R31.1

Commit message: add components and footprints
Parts:
- C37: footprint (none) -> 293D226X9035D2TE3:CAP_293D_D_VIS-M
- L1: footprint (none) -> VLS3012CX_100M_1:IND_VLS3012CX-100M-1
- R27: value R_US -> 1M47; footprint (none) -> Resistor_SMD:R_0402_1005Metric_Pad0.72x0.64mm_HandSolder
- R29: value R_US -> 71k5; footprint (none) -> Resistor_SMD:R_0402_1005Metric_Pad0.72x0.64mm_HandSolder
- R34, R35: footprint (none) -> Resistor_SMD:R_0402_1005Metric_Pad0.72x0.64mm_HandSolder
Changed lines of the file:
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@@
 			)
 		)
-		(property "Value" "R_US"
+		(property "Value" "71k5"
 			(at 153.67 64.7699 0)
 			(effects
@@
 			)
 		)
-		(property "Footprint" ""
+		(property "Footprint" "Resistor_SMD:R_0402_1005Metric_Pad0.72x0.64mm_HandSolder"
 			(at 152.146 63.754 90)
 			(effects
@@
 			)
 		)
-		(property "Value" "R_US"
+		(property "Value" "1M47"
 			(at 153.67 53.3399 0)
 			(effects
@@
 			)
 		)
-		(property "Footprint" ""
+		(property "Footprint" "Resistor_SMD:R_0402_1005Metric_Pad0.72x0.64mm_HandSolder"
 			(at 152.146 52.324 90)
 			(effects
@@
 			)
 		)
-		(property "Footprint" ""
+		(property "Footprint" "VLS3012CX_100M_1:IND_VLS3012CX-100M-1"
 			(at 127 30.48 0)
 			(effects
@@
 			)
 		)
-		(property "Footprint" ""
+		(property "Footprint" "293D226X9035D2TE3:CAP_293D_D_VIS-M"
 			(at 129.54 90.17 0)
 			(effects
@@
 			)
 		)
-		(property "Footprint" ""
+		(property "Footprint" "Resistor_SMD:R_0402_1005Metric_Pad0.72x0.64mm_HandSolder"
 			(at 112.776 87.884 90)
 			(effects
@@
 			)
 		)
-		(property "Footprint" ""
+		(property "Footprint" "Resistor_SMD:R_0402_1005Metric_Pad0.72x0.64mm_HandSolder"
 			(at 112.776 100.584 90)
 			(effects

Commit message: component placement for op amps
Connections:
- net 7V5_BUF1: now reaches R32.1, U12.1, U12.2 (-)
- net 7V5_IN: now reaches C27.1, R30.1, R31.2, U12.3 (+), U12.5 (+)
- net BST_FB: now reaches R27.2, R29.1, U11.3 (FB)
- net SW: now reaches L1.2, U11.1 (SW)
- net 7V5_BUF2: now reaches R33.1, U12.6 (-), U12.7
Other:
- note removed: "prob just put a 10u here or something."
Changed lines of the file:
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@@
-		)
-	)
-	(text "prob just put a 10u here or something."
-		(exclude_from_sim no)
-		(at 76.454 62.23 0)
-		(effects
-			(font
-				(size 1.27 1.27)
-			)
 		)
 	)
@@
 		)
 	)
+	(label "BST_FB"
+		(at 139.7 58.42 0)
+		(fields_autoplaced yes)
+		(effects
+			(font
+				(size 1.27 1.27)
+			)
+			(justify left bottom)
+		)
+	)
+	(label "7V5_BUF2"
+		(at 91.44 166.37 0)
+		(fields_autoplaced yes)
+		(effects
+			(font
+				(size 1.27 1.27)
+			)
+			(justify left bottom)
+		)
+	)
+	(label "7V5_BUF1"
+		(at 91.44 142.24 0)
+		(fields_autoplaced yes)
+		(effects
+			(font
+				(size 1.27 1.27)
+			)
+			(justify left bottom)
+		)
+	)
+	(label "7V5_IN"
+		(at 71.12 132.08 0)
+		(fields_autoplaced yes)
+		(effects
+			(font
+				(size 1.27 1.27)
+			)
+			(justify left bottom)
+		)
+	)
 	(label "ADJ"
 		(at 106.68 93.98 0)
 		(fields_autoplaced yes)
 		(effects
+			(font
+				(size 1.27 1.27)
+			)
+			(justify left bottom)
+		)
+	)
+	(label "SW"
+		(at 137.16 43.18 0)
+		(fields_autoplaced yes)
+		(effects

Commit message: complete layout
Parts:
- U13: footprint LM2941:DFN400X400X80-9N -> LM2941:NGN0008A
Changed lines of the file:
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@@
 			)
 		)
-		(property "Footprint" "LM2941:DFN400X400X80-9N"
+		(property "Footprint" "LM2941:NGN0008A"
 			(at 90.17 88.9 0)
 			(effects
