File: DacAmp/DacAmp.kicad_pcb (KiCad board)
At the start: 4 copper layers, 92 x 70.5 mm, 111 parts, among them J1 AudioPlug3, J2 USB_B, U1 PCM2906C, U10 TLV70237_SOT23-5, U11 TLV61046ADB, U12 NE5532, U13 LM2941LD_NOPB, U2 NE5532, U3 NE5532, U4 NE5532, U5 NE5532, U6 NE5532, U7 NE5532, U8 NE5532, U9 NE5532, Y1 12MHz

Commit message: update release 1
Routing:
- net GND: vias 499 -> 503
Other:
- board text added: "USB Headphone Amplifier Uzair Syed November 2024 Revision -"
Changed lines of the file:
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@@
 		(layer "Edge.Cuts")
 	)
+	(gr_text "USB Headphone Amplifier\nUzair Syed\nNovember 2024\nRevision -"
+		(at 132.7374 103.2974 0)
+		(layer "F.SilkS")
+		(effects
+			(font
+				(size 1.5 1.5)
+				(thickness 0.153)
+			)
+			(justify left bottom)
+		)
+	)
 	(segment
 		(start 170.6145 48.2146)
@@
 	)
 	(via
+		(at 147.3424 50.5924)
+		(size 0.6)
+		(drill 0.4)
+		(layers "F.Cu" "B.Cu")
+		(free yes)
+		(net 2)
+	)
+	(via
 		(at 149.8824 67.7374)
 		(size 0.6)
@@
 	)
 	(via
+		(at 163.8524 49.9574)
+		(size 0.6)
+		(drill 0.4)
+		(layers "F.Cu" "B.Cu")
+		(free yes)
+		(net 2)
+	)
+	(via
 		(at 147.3424 85.5174)
 		(size 0.6)
@@
 	)
 	(via
+		(at 145.4374 50.5924)
+		(size 0.6)
+		(drill 0.4)
+		(layers "F.Cu" "B.Cu")
+		(free yes)
+		(net 2)
+	)
+	(via
 		(at 157.5024 67.7374)
 		(size 0.6)
@@
 	)
 	(via
+		(at 167.051453 46.116002)
+		(size 0.6)
+		(drill 0.4)
+		(layers "F.Cu" "B.Cu")
+		(free yes)
+		(net 2)
+	)
+	(via
 		(at 121.9424 62.0224)
 		(size 0.6)
@@
 		(polygon
 			(pts
-				(xy 138.8228 46.7956) (xy 133.8952 46.7956) (xy 133.8952 50.8596) (xy 140.0724 52.9624) (xy 148.4224 52.9624)
+				(xy 138.8228 46.7956) (xy 133.8952 46.7956) (xy 133.8952 50.8596) (xy 135.2774 52.9624) (xy 148.4224 52.9624)
 				(xy 148.5724 52.8124) (xy 148.5724 52.0624) (xy 148.4224 51.9124) (xy 140.0224 51.9124) (xy 138.8228 50.8596)
 			)
